File: g1-ata-25.sch (KiCad schematic (older format))
At the start: 30 parts, among them P1 G1_DC_SOCKET, P2 G1_GD_PLUGNH, P3 IDE_40PIN, P4 IDE_44PIN, P5 CONN_01X02, P6 CONN_01X04, P7 CONN_01X04, P8 CONN_01X05, U1 TCXO_DFAS11, U2 TS30011-M050

Commit message: Added fuse + polarity protection for 5V input (not yet routed).
Parts:
- removed U1: TCXO_DFAS11, doragasu:OSC_F530L, symbol TCXO_DFAS11
- added D3: D, Diodes_SMD:MiniMELF_Standard, symbol D
- added F2: F_Small, Capacitors_SMD:C_0805, symbol F_Small
- added U1: DSC1001, doragasu:DSC1001-32x25M, symbol DSC1001
- F1: manf# (none) -> MFU0805FF02000P100
- L1: footprint Capacitors_SMD:C_1206 -> doragasu:INDUCTOR-NR4018; manf# (none) -> NR4018T4R7M
- renumbered JP5 to JP3, JP3 to JP4, JP4 to JP5
Connections:
- net +3V3: now also U1.1 (~STBY), U1.4 (VDD)
- net GND: now also JP1.1, D3.2 (A), U1.2 (GND)
- net at P1.B23 (CDDA_CLK): no longer JP1.1
- net at JP1.3: now also U1.3 (OUT)
- net at P7.4 (P4): now also F2.1; no longer JP3.1
- new net: D3.1 (K), F2.2, JP3.1
Other:
- moved on the sheet: C8, JP1
Changed lines of the file:
@@
 $EndDescr
-$Comp
-L TCXO_DFAS11 U1
-U 1 1 574BD61B
-P 2450 4950
-F 0 "U1" H 2450 5365 50  0000 C CNN
-F 1 "TCXO_DFAS11" H 2450 5274 50  0000 C CNN
-F 2 "doragasu:OSC_F530L" H 2450 4950 50  0001 C CNN
-F 3 "" H 2450 4950 50  0000 C CNN
-	1    2450 4950
-	1    0    0    -1
-$EndComp
 $Comp
 L GND #PWR01
@@
 L +3.3V #PWR019
 U 1 1 574C7B76
-P 1750 4800
-F 0 "#PWR019" H 1750 4650 50  0001 C CNN
-F 1 "+3.3V" H 1750 4950 50  0000 C CNN
-F 2 "" H 1750 4800 50  0000 C CNN
-F 3 "" H 1750 4800 50  0000 C CNN
-	1    1750 4800
+P 2100 4800
+F 0 "#PWR019" H 2100 4650 50  0001 C CNN
+F 1 "+3.3V" H 2100 4950 50  0000 C CNN
+F 2 "" H 2100 4800 50  0000 C CNN
+F 3 "" H 2100 4800 50  0000 C CNN
+	1    2100 4800
 	1    0    0    -1
 $EndComp
@@
 L GND #PWR020
 U 1 1 574C7F12
-P 3150 5100
-F 0 "#PWR020" H 3150 4850 50  0001 C CNN
-F 1 "GND" H 3155 4927 50  0001 C CNN
-F 2 "" H 3150 5100 50  0000 C CNN
-F 3 "" H 3150 5100 50  0000 C CNN
-	1    3150 5100
+P 3100 5100
+F 0 "#PWR020" H 3100 4850 50  0001 C CNN
+F 1 "GND" H 3105 4927 50  0001 C CNN
+F 2 "" H 3100 5100 50  0000 C CNN
+F 3 "" H 3100 5100 50  0000 C CNN
+	1    3100 5100
 	1    0    0    -1
 $EndComp
@@
 L JUMPER3 JP1
 U 1 1 574C8107
-P 3150 4200
-F 0 "JP1" V 3104 4301 50  0000 L CNN
-F 1 "JUMPER3" V 3195 4301 50  0001 L CNN
-F 2 "Pin_Headers:Pin_Header_Straight_1x03" H 3150 4200 50  0001 C CNN
-F 3 "" H 3150 4200 50  0000 C CNN
-F 4 "CDDA CLK SEL" V 3200 4650 60  0000 C CNN "Func"
-	1    3150 4200
+P 3100 4200
+F 0 "JP1" V 3054 4301 50  0000 L CNN
+F 1 "JUMPER3" V 3145 4301 50  0001 L CNN
+F 2 "Pin_Headers:Pin_Header_Straight_1x03" H 3100 4200 50  0001 C CNN
+F 3 "" H 3100 4200 50  0000 C CNN
+F 4 "CDDA CLK SEL" V 3150 4650 60  0000 C CNN "Func"
+	1    3100 4200
 	0    -1   1    0
 $EndComp
@@
 F 0 "L1" V 7916 5100 50  0000 C CNN
 F 1 "4.7u" V 7825 5100 50  0000 C CNN
-F 2 "Capacitors_SMD:C_1206" H 7700 5100 50  0001 C CNN
+F 2 "doragasu:INDUCTOR-NR4018" H 7700 5100 50  0001 C CNN
 F 3 "" H 7700 5100 50  0000 C CNN
+F 4 "NR4018T4R7M" V 7700 5100 60  0001 C CNN "manf#"
 	1    7700 5100
 	0    -1   -1   0
@@
 NoConn ~ 7050 5700
 $Comp
-L JUMPER3 JP3
+L JUMPER3 JP4
 U 1 1 574CB39F
 P 8900 4750
-F 0 "JP3" V 8800 4850 50  0000 L CNN
+F 0 "JP4" V 8800 4850 50  0000 L CNN
 F 1 "JUMPER3" V 8945 4851 50  0001 L CNN
 F 2 "Pin_Headers:Pin_Header_Straight_1x03" H 8900 4750 50  0001 C CNN
@@
 F 2 "Capacitors_SMD:C_0805" H 4200 4600 50  0001 C CNN
 F 3 "" H 4200 4600 50  0000 C CNN
+F 4 "MFU0805FF02000P100" H 4200 4600 60  0001 C CNN "manf#"
 	1    4200 4600
 	1    0    0    -1
@@
 L C C8
 U 1 1 574D76B9
-P 2450 5600
-F 0 "C8" H 2565 5646 50  0000 L CNN
-F 1 "100n" H 2565 5555 50  0000 L CNN
-F 2 "Capacitors_SMD:C_0805" H 2488 5450 50  0001 C CNN
-F 3 "" H 2450 5600 50  0000 C CNN
-	1    2450 5600
+P 2600 5600
+F 0 "C8" H 2715 5646 50  0000 L CNN
+F 1 "100n" H 2715 5555 50  0000 L CNN
+F 2 "Capacitors_SMD:C_0805" H 2638 5450 50  0001 C CNN
+F 3 "" H 2600 5600 50  0000 C CNN
+	1    2600 5600
 	1    0    0    -1
 $EndComp
@@
 L +3.3V #PWR035
 U 1 1 574D7890
-P 2450 5450
-F 0 "#PWR035" H 2450 5300 50  0001 C CNN
-F 1 "+3.3V" H 2450 5600 50  0000 C CNN
-F 2 "" H 2450 5450 50  0000 C CNN
-F 3 "" H 2450 5450 50  0000 C CNN
-	1    2450 5450
+P 2600 5450
+F 0 "#PWR035" H 2600 5300 50  0001 C CNN
+F 1 "+3.3V" H 2600 5600 50  0000 C CNN
+F 2 "" H 2600 5450 50  0000 C CNN
+F 3 "" H 2600 5450 50  0000 C CNN
+	1    2600 5450
 	1    0    0    -1
 $EndComp
@@
 L GND #PWR036
 U 1 1 574D7923
-P 2450 5750
-F 0 "#PWR036" H 2450 5500 50  0001 C CNN
-F 1 "GND" H 2455 5577 50  0001 C CNN
-F 2 "" H 2450 5750 50  0000 C CNN
-F 3 "" H 2450 5750 50  0000 C CNN
-	1    2450 5750
+P 2600 5750
+F 0 "#PWR036" H 2600 5500 50  0001 C CNN
+F 1 "GND" H 2605 5577 50  0001 C CNN
+F 2 "" H 2600 5750 50  0000 C CNN
+F 3 "" H 2600 5750 50  0000 C CNN
+	1    2600 5750
 	1    0    0    -1
 $EndComp
@@
 ~IDE_CS1
 $Comp
-L JUMPER JP4
+L JUMPER JP5
 U 1 1 574E24DB
 P 10300 4850
-F 0 "JP4" H 10300 5129 50  0000 C CNN
+F 0 "JP5" H 10300 5129 50  0000 C CNN
 F 1 "JUMPER" H 10300 5023 50  0001 C CNN
 F 2 "Pin_Headers:Pin_Header_Straight_1x02" H 10300 4850 50  0001 C CNN
@@
 	5400 5300 5450 5300
 Wire Wire Line
-	3150 3550 3150 3950
-Wire Wire Line
 	5700 3550 5250 3550
 Wire Wire Line
 	5700 4200 5700 3550
 Wire Wire Line
-	3250 4200 5700 4200
-Wire Wire Line
-	2650 3550 3150 3550
-Wire Wire Line
-	3150 4450 3150 4800
-Connection ~ 1750 4800
-Wire Wire Line
-	1750 5100 1750 4800
+	3200 4200 5700 4200
+Wire Wire Line
+	3100 4450 3100 4800
+Connection ~ 2100 4800
+Wire Wire Line
+	2100 5100 2100 4800
 Wire Wire Line
 	10550 3350 10450 3350
@@
 Connection ~ 4050 4800
 Wire Wire Line
-	3950 4900 3950 5000
-Wire Wire Line
-	3950 5000 3500 5000
-Wire Wire Line
-	3500 5000 3500 4300
+	3500 5650 3500 4300
 Wire Wire Line
 	3500 4300 8600 4300
 $Comp
-L JUMPER3 JP5
+L JUMPER3 JP3
 U 1 1 575912D5
 P 8600 4750
-F 0 "JP5" V 8500 4850 50  0000 L CNN
+F 0 "JP3" V 8500 4850 50  0000 L CNN
 F 1 "JUMPER3" V 8645 4851 50  0001 L CNN
 F 2 "Pin_Headers:Pin_Header_Straight_1x03" H 8600 4750 50  0001 C CNN
@@
 Wire Wire Line
 	8750 4750 8700 4750
+$Comp
+L DSC1001 U1
+U 1 1 57595987
+P 2600 4950
+F 0 "U1" H 2600 5365 50  0000 C CNN
+F 1 "DSC1001" H 2600 5274 50  0000 C CNN
+F 2 "doragasu:DSC1001-32x25M" H 2600 4950 50  0001 C CNN
+F 3 "" H 2600 4950 50  0000 C CNN
+	1    2600 4950
+	1    0    0    -1
+$EndComp
+Wire Wire Line
+	2700 3550 3100 3550
+Wire Wire Line
+	3100 3550 3100 3950
+Connection ~ 2700 3550
+$Comp
+L F_Small F2
+U 1 1 57599F7E
+P 4200 5200
+F 0 "F2" H 4200 5293 50  0000 C CNN
+F 1 "F_Small" H 4200 5294 50  0001 C CNN
+F 2 "Capacitors_SMD:C_0805" H 4200 5200 50  0001 C CNN
+F 3 "" H 4200 5200 50  0000 C CNN
+F 4 "MFU0805FF02000P100" H 4200 5200 60  0001 C CNN "manf#"
+	1    4200 5200
+	1    0    0    -1
+$EndComp
+$Comp
+L D D3
+U 1 1 5759A055
+P 4350 5350
+F 0 "D3" V 4304 5428 50  0000 L CNN
+F 1 "D" V 4395 5428 50  0000 L CNN
+F 2 "Diodes_SMD:MiniMELF_Standard" H 4350 5350 50  0001 C CNN
+F 3 "" H 4350 5350 50  0000 C CNN
+	1    4350 5350
+	0    1    1    0
+$EndComp
+Wire Wire Line
+	3950 4900 3950 5200
+Wire Wire Line
+	3950 5200 4100 5200
+Wire Wire Line
+	4300 5200 4600 5200
+$Comp
+L GND #PWR044
+U 1 1 5759A3FB
+P 4350 5500
+F 0 "#PWR044" H 4350 5250 50  0001 C CNN
+F 1 "GND" H 4355 5327 50  0001 C CNN
+F 2 "" H 4350 5500 50  0000 C CNN
+F 3 "" H 4350 5500 50  0000 C CNN
+	1    4350 5500
+	1    0    0    -1
+$EndComp
+Wire Wire Line
+	4600 5200 4600 5650
+Wire Wire Line
+	4600 5650 3500 5650
+Connection ~ 4350 5200
 $EndSCHEMATC

Commit message: Added bootstrap capacitor value.
Parts:
- C5: value C -> 22n
Changed lines of the file:
@@
 LIBS:Oscillators
 LIBS:g1-ata-25-cache
-EELAYER 25 0
+EELAYER 26 0
 EELAYER END
 $Descr A4 11693 8268
@@
 P 7250 4950
 F 0 "C5" H 7365 4996 50  0000 L CNN
-F 1 "C" H 7365 4905 50  0000 L CNN
+F 1 "22n" H 7365 4905 50  0000 L CNN
 F 2 "Capacitors_SMD:C_0805" H 7288 4800 50  0001 C CNN
 F 3 "" H 7250 4950 50  0000 C CNN

Commit message: Fixed connection to pass CDDA_CLK from GD-ROM drive.
Parts:
- U1: manf# (none) -> DSC1001CE1-033.8688T
Connections:
- net +5V: now also D1.2 (A)
- net GND: no longer JP1.1
- net at P1.B23 (CDDA_CLK): now also JP1.1
- net at P5.1 (P1), R1.1: now also D1.1 (K)
Changed lines of the file:
@@
 	7000 3750 7000 4100
 Wire Wire Line
-	7000 4100 6950 4100
+	7000 4100 6900 4100
 Wire Wire Line
 	7300 4100 7500 4100
@@
 F 2 "doragasu:DSC1001-32x25M" H 2600 4950 50  0001 C CNN
 F 3 "" H 2600 4950 50  0000 C CNN
+F 4 "DSC1001CE1-033.8688T" H 2600 4950 60  0001 C CNN "manf#"
 	1    2600 4950
 	1    0    0    -1
 $EndComp
 Wire Wire Line
-	2700 3550 3100 3550
-Wire Wire Line
 	3100 3550 3100 3950
-Connection ~ 2700 3550
 $Comp
 L F_Small F2
@@
 	4600 5650 3500 5650
 Connection ~ 4350 5200
+Wire Wire Line
+	6550 4100 6600 4100
+Wire Wire Line
+	3100 3550 2650 3550
 $EndSCHEMATC
